File: rpi.kicad_sch (KiCad schematic)
At the start: 9 parts, among them U2 RaspberryPi-4/5, U701 24LC32AT-x/OT

Commit message: fixed some stuff
Connections:
- no-connect marks 17 -> 18
Changed lines of the file:
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@@
+	)
+	(no_connect
+		(at 137.16 83.82)
 	)
 	(no_connect
