File: ethernet.kicad_sch (KiCad schematic)
At the start: 34 parts, among them J5 Ethernet, U601 KSZ8851-16MLL, U602 93LC46B/SN

Commit message: fixed some stuff
Parts:
- R601: value 10k -> 1k
Changed lines of the file:
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@@
 			)
 		)
-		(property "Value" "10k"
+		(property "Value" "1k"
 			(at 71.12 95.2499 0)
 			(effects

Commit message: some changes in schematic and added pcb
Parts:
- L601, L602, L603: footprint Inductor_SMD:L_0603_1608Metric -> Inductor_SMD:L_0805_2012Metric
Changed lines of the file:
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@@
 			)
 		)
-		(property "Footprint" "Inductor_SMD:L_0603_1608Metric"
+		(property "Footprint" "Inductor_SMD:L_0805_2012Metric"
 			(at 261.62 96.52 0)
 			(effects
@@
 			)
 		)
-		(property "Footprint" "Inductor_SMD:L_0603_1608Metric"
+		(property "Footprint" "Inductor_SMD:L_0805_2012Metric"
 			(at 139.7 73.66 0)
 			(effects
@@
 			)
 		)
-		(property "Footprint" "Inductor_SMD:L_0603_1608Metric"
+		(property "Footprint" "Inductor_SMD:L_0805_2012Metric"
 			(at 66.04 40.64 0)
 			(effects
