File: fpga_misc.kicad_sch (KiCad schematic)
At the start: 32 parts, among them J10 JTAG, U1 XC6SLX9-TQG144, U101 LM809, U102 W25Q16JVSn, U103 ASDMB-xxxMHz

Commit message: fixed some stuff
Parts:
- U103: value ASDMB-xxxMHz -> ASDMB-50MHz
Changed lines of the file:
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@@
 			)
 		)
-		(property "Value" "ASDMB-xxxMHz"
+		(property "Value" "ASDMB-50MHz"
 			(at 257.81 29.21 0)
 			(effects

Commit message: some changes in schematic and added pcb
Parts:
- J10: now left out of the parts list
Changed lines of the file:
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@@
 		(unit 1)
 		(exclude_from_sim no)
-		(in_bom yes)
+		(in_bom no)
 		(on_board yes)
 		(dnp no)
