File: stmbl-fpga-master.kicad_pcb (KiCad board)
At the start: 4 copper layers, 99.8 x 99.8 mm, 280 parts, among them J1 POWER, J10 JTAG, J2 OUT, J3 IN, J4 Parallel expansion port, J5 Ethernet, J6 8P8C_x4, J7 8P8C_x4, J8 8P8C_x4, J9 8P8C_x2, Q101 AO3400A, Q2401 SS8550, U1 XC6SLX9-TQG144, U1001 SP3485EN, U1002 SP3485EN, U101 LM809, U102 W25Q16JVSn, U103 ASDMB-50MHz, U1101 SP3485EN, U1102 SP3485EN, U1201 SP3485EN, U1202 SP3485EN, U1301 SP3485EN, U1302 SP3485EN, U1401 SP3485EN, U1402 SP3485EN, U1501 SP3485EN, U1502 SP3485EN, U1601 SP3485EN, U1602 SP3485EN, U1701 SP3485EN, U1702 SP3485EN, U1801 SP3485EN, U1802 SP3485EN, U1901 SP3485EN, U1902 SP3485EN, U2 RaspberryPi-4/5, U2001 SP3485EN, U2002 SP3485EN, U201 TPS56637RPAR, U202 TPS56637RPAR, U203 AZ1117-3.3, U204 AZ1117-1.2, U2101 SP3485EN, U2102 SP3485EN, U2201 SP3485EN, U2202 SP3485EN, U2301 SP3485EN, U2302 SP3485EN, U2401 74CB3T16210DGG, U601 KSZ8851-16MLL, U602 93LC46B/SN, U701 24LC32AT-x/OT

Commit message: some changes in schematic and added pcb
Parts:
- added REF**: JLC_Tooling_Hole, stmbl-fpga-master:JLC_Tooling_Hole, F.Cu at (32.5, 31.0)
- added REF**: JLC_Tooling_Hole, stmbl-fpga-master:JLC_Tooling_Hole, F.Cu at (122.5, 31.0)
- added REF**: JLC_Tooling_Hole, stmbl-fpga-master:JLC_Tooling_Hole, F.Cu at (127.0, 128.8)
- L601, L602, L603: footprint Inductor_SMD:L_0603_1608Metric -> Inductor_SMD:L_0805_2012Metric
- moved L603 0.36 mm to (83.8, 37.4)
- moved L602 0.33 mm to (77.5, 51.6)
- moved L601 0.27 mm to (72.9, 46.8)
Routing:
- net GND: track 537.0 -> 537.7 mm
Other:
- board text added: "JLCJLCJLCJLC"
